File: lm324.brd (EAGLE design)
At the start: 160 x 100 mm, 15 parts, among them IC1 LM324N

Commit message: BRD2
Parts:
- moved R7 17.1 mm to (40.5, 30.7), turned to 180 degrees
- moved R8 8.89 mm to (56.7, 32.4), turned to 180 degrees
- moved R6 7.76 mm to (45.5, 30.7)
- moved R1 5.76 mm to (45.6, 27.6), turned to 0 degrees
- moved R3 4.22 mm to (40.5, 27.6), turned to 180 degrees
- moved JP3 2.98 mm to (34.9, 21.6)
- moved JP2 2.75 mm to (65.6, 16.8)
- moved C1 2.60 mm to (45.6, 24.5)
- moved R2 2.36 mm to (40.4, 24.5)
- moved C2 1.17 mm to (52.4, 29.2)
- moved C3 1.15 mm to (61.2, 29.1)
- moved R5 0.33 mm to (55.1, 16.9)
- moved R4 0.31 mm to (50.4, 16.8)
Routing:
- net GND: track 0.00 -> 102.9 mm
- net N$7: track 0.00 -> 37.0 mm
- net 5V: track 0.00 -> 25.7 mm
- net N$1: track 0.00 -> 24.6 mm
- net N$8: track 0.00 -> 22.5 mm
- net N$4: track 0.00 -> 20.8 mm
- net N$6: track 0.00 -> 15.4 mm
- net N$2: track 0.00 -> 7.14 mm
- net N$5: track 0.00 -> 3.12 mm
