File: lm324.brd (EAGLE design)
At the start: 160 x 100 mm, 15 parts, among them IC1 LM324N

Commit message: Rate R6 & R5
Parts:
- R5: value 100k -> 20k
- R6: value 10k -> 50k
Changed lines of the file:
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@@
 <element name="C1" library="resistor" package="C0805" value="0.01u" x="45.61" y="24.49" rot="MR180"/>
 <element name="R4" library="resistor" package="R0805" value="100k" x="50.4" y="16.77" rot="MR0"/>
-<element name="R5" library="resistor" package="R0805" value="100k" x="55.09" y="16.86" rot="MR0"/>
+<element name="R5" library="resistor" package="R0805" value="20k" x="55.09" y="16.86" rot="MR0"/>
 <element name="C2" library="resistor" package="E3,5-8" value="10u" x="52.35" y="29.24" rot="R90"/>
-<element name="R6" library="resistor" package="R0805" value="10k" x="45.55" y="30.67" rot="MR180"/>
+<element name="R6" library="resistor" package="R0805" value="50k" x="45.55" y="30.67" rot="MR180"/>
 <element name="R7" library="resistor" package="R0805" value="6.2k" x="40.49" y="30.69" rot="MR180"/>
 <element name="R8" library="resistor" package="R0805" value="10k" x="56.69" y="32.42" rot="MR180"/>
