File: lm324.sch (EAGLE design)
At the start: 15 parts, among them IC1 LM324N

Commit message: Rate R6 & R5
Parts:
- R5: value 100k -> 20k
- R6: value 10k -> 50k
Changed lines of the file:
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@@
 <part name="GND1" library="supply1" deviceset="GND" device=""/>
 <part name="R4" library="resistor" deviceset="R-EU_" device="R0805" value="100k"/>
-<part name="R5" library="resistor" deviceset="R-EU_" device="R0805" value="100k"/>
+<part name="R5" library="resistor" deviceset="R-EU_" device="R0805" value="20k"/>
 <part name="C2" library="resistor" deviceset="CPOL-EU" device="E3.5-8" value="10u"/>
-<part name="R6" library="resistor" deviceset="R-EU_" device="R0805" value="10k"/>
+<part name="R6" library="resistor" deviceset="R-EU_" device="R0805" value="50k"/>
 <part name="R7" library="resistor" deviceset="R-EU_" device="R0805" value="6.2k"/>
 <part name="R8" library="resistor" deviceset="R-EU_" device="R0805" value="10k"/>
